Commit message: FIX: PM01'S torque limit is wrong

File: engineai_gym/engineai_gym/resources/robots/biped/pm01/urdf/pm01.urdf (robot description, URDF)
Before this commit: robot pm01, 25 links, 24 joints
Joints:
- joint j02_hip_yaw_l: limit lower=-1.57 upper=4.014 effort=61 velocity=35.2 -> lower=-1.57 upper=4.014 effort=52 velocity=35.2
- joint j04_ankle_pitch_l: limit lower=-0.6807 upper=0.7243 effort=61 velocity=35.2 -> lower=-0.6807 upper=0.7243 effort=52 velocity=35.2
- joint j05_ankle_roll_l: limit lower=-0.2618 upper=0.2618 effort=61 velocity=35.2 -> lower=-0.2618 upper=0.2618 effort=52 velocity=35.2
- joint j08_hip_yaw_r: limit lower=-4.014 upper=1.57 effort=61 velocity=35.2 -> lower=-4.014 upper=1.57 effort=52 velocity=35.2
- joint j10_ankle_pitch_r: limit lower=-0.6807 upper=0.7243 effort=61 velocity=35.2 -> lower=-0.6807 upper=0.7243 effort=52 velocity=35.2
- joint j11_ankle_roll_r: limit lower=-0.2618 upper=0.2618 effort=61 velocity=35.2 -> lower=-0.2618 upper=0.2618 effort=52 velocity=35.2
- joint j12_waist_yaw: limit lower=-4.014 upper=1.57 effort=61 velocity=35.2 -> lower=-4.014 upper=1.57 effort=52 velocity=35.2
- joint j13_shoulder_pitch_l: limit lower=-2.9671 upper=2.7925 effort=61 velocity=35.2 -> lower=-2.9671 upper=2.7925 effort=52 velocity=35.2
- joint j14_shoulder_roll_l: limit lower=-0.6108 upper=2.3562 effort=61 velocity=35.2 -> lower=-0.6108 upper=2.3562 effort=52 velocity=35.2
- joint j15_shoulder_yaw_l: limit lower=-2.618 upper=2.618 effort=61 velocity=35.2 -> lower=-2.618 upper=2.618 effort=52 velocity=35.2
- joint j16_elbow_pitch_l: limit lower=-2.1948 upper=0.7374 effort=61 velocity=35.2 -> lower=-2.1948 upper=0.7374 effort=52 velocity=35.2
- joint j17_elbow_yaw_l: limit lower=-2.618 upper=2.618 effort=61 velocity=35.2 -> lower=-2.618 upper=2.618 effort=52 velocity=35.2
- joint j18_shoulder_pitch_r: limit lower=-2.9671 upper=2.7925 effort=61 velocity=35.2 -> lower=-2.9671 upper=2.7925 effort=52 velocity=35.2
- joint j19_shoulder_roll_r: limit lower=-2.3562 upper=0.6108 effort=61 velocity=35.2 -> lower=-2.3562 upper=0.6108 effort=52 velocity=35.2
- joint j20_shoulder_yaw_r: limit lower=-2.618 upper=2.618 effort=61 velocity=35.2 -> lower=-2.618 upper=2.618 effort=52 velocity=35.2
- joint j21_elbow_pitch_r: limit lower=-2.1948 upper=0.7374 effort=61 velocity=35.2 -> lower=-2.1948 upper=0.7374 effort=52 velocity=35.2
- joint j22_elbow_yaw_r: limit lower=-2.618 upper=2.618 effort=61 velocity=35.2 -> lower=-2.618 upper=2.618 effort=52 velocity=35.2
- joint j23_head_yaw: limit lower=-0.6109 upper=0.6109 effort=61 velocity=35.2 -> lower=-0.6109 upper=0.6109 effort=52 velocity=35.2

File: engineai_gym/engineai_gym/resources/robots/biped/pm01/urdf/pm01_only_legs.urdf (robot description, URDF)
Before this commit: robot pm01, 25 links, 24 joints
Joints:
- joint j02_hip_yaw_l: limit lower=-1.57 upper=4.014 effort=61 velocity=35.2 -> lower=-1.57 upper=4.014 effort=52 velocity=35.2
- joint j04_ankle_pitch_l: limit lower=-0.6807 upper=0.7243 effort=61 velocity=35.2 -> lower=-0.6807 upper=0.7243 effort=52 velocity=35.2
- joint j05_ankle_roll_l: limit lower=-0.2618 upper=0.2618 effort=61 velocity=35.2 -> lower=-0.2618 upper=0.2618 effort=52 velocity=35.2
- joint j08_hip_yaw_r: limit lower=-4.014 upper=1.57 effort=61 velocity=35.2 -> lower=-4.014 upper=1.57 effort=52 velocity=35.2
- joint j10_ankle_pitch_r: limit lower=-0.6807 upper=0.7243 effort=61 velocity=35.2 -> lower=-0.6807 upper=0.7243 effort=52 velocity=35.2
- joint j11_ankle_roll_r: limit lower=-0.2618 upper=0.2618 effort=61 velocity=35.2 -> lower=-0.2618 upper=0.2618 effort=52 velocity=35.2
- joint j12_waist_yaw: limit lower=-4.014 upper=1.57 effort=61 velocity=35.2 -> lower=-4.014 upper=1.57 effort=52 velocity=35.2
- joint j13_shoulder_pitch_l: limit lower=-2.9671 upper=2.7925 effort=61 velocity=35.2 -> lower=-2.9671 upper=2.7925 effort=52 velocity=35.2
- joint j14_shoulder_roll_l: limit lower=-0.6108 upper=2.3562 effort=61 velocity=35.2 -> lower=-0.6108 upper=2.3562 effort=52 velocity=35.2
- joint j15_shoulder_yaw_l: limit lower=-2.618 upper=2.618 effort=61 velocity=35.2 -> lower=-2.618 upper=2.618 effort=52 velocity=35.2
- joint j16_elbow_pitch_l: limit lower=-2.1948 upper=0.7374 effort=61 velocity=35.2 -> lower=-2.1948 upper=0.7374 effort=52 velocity=35.2
- joint j17_elbow_yaw_l: limit lower=-2.618 upper=2.618 effort=61 velocity=35.2 -> lower=-2.618 upper=2.618 effort=52 velocity=35.2
- joint j18_shoulder_pitch_r: limit lower=-2.9671 upper=2.7925 effort=61 velocity=35.2 -> lower=-2.9671 upper=2.7925 effort=52 velocity=35.2
- joint j19_shoulder_roll_r: limit lower=-2.3562 upper=0.6108 effort=61 velocity=35.2 -> lower=-2.3562 upper=0.6108 effort=52 velocity=35.2
- joint j20_shoulder_yaw_r: limit lower=-2.618 upper=2.618 effort=61 velocity=35.2 -> lower=-2.618 upper=2.618 effort=52 velocity=35.2
- joint j21_elbow_pitch_r: limit lower=-2.1948 upper=0.7374 effort=61 velocity=35.2 -> lower=-2.1948 upper=0.7374 effort=52 velocity=35.2
- joint j22_elbow_yaw_r: limit lower=-2.618 upper=2.618 effort=61 velocity=35.2 -> lower=-2.618 upper=2.618 effort=52 velocity=35.2
- joint j23_head_yaw: limit lower=-0.6109 upper=0.6109 effort=61 velocity=35.2 -> lower=-0.6109 upper=0.6109 effort=52 velocity=35.2

File: engineai_gym/engineai_gym/resources/robots/biped/pm01/urdf/pm01_only_legs_simple_collision.urdf (robot description, URDF)
Before this commit: robot pm01, 25 links, 24 joints
Joints:
- joint j02_hip_yaw_l: limit lower=-1.57 upper=4.014 effort=61 velocity=35.2 -> lower=-1.57 upper=4.014 effort=52 velocity=35.2
- joint j04_ankle_pitch_l: limit lower=-0.6807 upper=0.7243 effort=61 velocity=35.2 -> lower=-0.6807 upper=0.7243 effort=52 velocity=35.2
- joint j05_ankle_roll_l: limit lower=-0.2618 upper=0.2618 effort=61 velocity=35.2 -> lower=-0.2618 upper=0.2618 effort=52 velocity=35.2
- joint j08_hip_yaw_r: limit lower=-4.014 upper=1.57 effort=61 velocity=35.2 -> lower=-4.014 upper=1.57 effort=52 velocity=35.2
- joint j10_ankle_pitch_r: limit lower=-0.6807 upper=0.7243 effort=61 velocity=35.2 -> lower=-0.6807 upper=0.7243 effort=52 velocity=35.2
- joint j11_ankle_roll_r: limit lower=-0.2618 upper=0.2618 effort=61 velocity=35.2 -> lower=-0.2618 upper=0.2618 effort=52 velocity=35.2
- joint j12_waist_yaw: limit lower=-4.014 upper=1.57 effort=61 velocity=35.2 -> lower=-4.014 upper=1.57 effort=52 velocity=35.2
- joint j13_shoulder_pitch_l: limit lower=-2.9671 upper=2.7925 effort=61 velocity=35.2 -> lower=-2.9671 upper=2.7925 effort=52 velocity=35.2
- joint j14_shoulder_roll_l: limit lower=-0.6108 upper=2.3562 effort=61 velocity=35.2 -> lower=-0.6108 upper=2.3562 effort=52 velocity=35.2
- joint j15_shoulder_yaw_l: limit lower=-2.618 upper=2.618 effort=61 velocity=35.2 -> lower=-2.618 upper=2.618 effort=52 velocity=35.2
- joint j16_elbow_pitch_l: limit lower=-2.1948 upper=0.7374 effort=61 velocity=35.2 -> lower=-2.1948 upper=0.7374 effort=52 velocity=35.2
- joint j17_elbow_yaw_l: limit lower=-2.618 upper=2.618 effort=61 velocity=35.2 -> lower=-2.618 upper=2.618 effort=52 velocity=35.2
- joint j18_shoulder_pitch_r: limit lower=-2.9671 upper=2.7925 effort=61 velocity=35.2 -> lower=-2.9671 upper=2.7925 effort=52 velocity=35.2
- joint j19_shoulder_roll_r: limit lower=-2.3562 upper=0.6108 effort=61 velocity=35.2 -> lower=-2.3562 upper=0.6108 effort=52 velocity=35.2
- joint j20_shoulder_yaw_r: limit lower=-2.618 upper=2.618 effort=61 velocity=35.2 -> lower=-2.618 upper=2.618 effort=52 velocity=35.2
- joint j21_elbow_pitch_r: limit lower=-2.1948 upper=0.7374 effort=61 velocity=35.2 -> lower=-2.1948 upper=0.7374 effort=52 velocity=35.2
- joint j22_elbow_yaw_r: limit lower=-2.618 upper=2.618 effort=61 velocity=35.2 -> lower=-2.618 upper=2.618 effort=52 velocity=35.2
- joint j23_head_yaw: limit lower=-0.6109 upper=0.6109 effort=61 velocity=35.2 -> lower=-0.6109 upper=0.6109 effort=52 velocity=35.2

File: engineai_gym/engineai_gym/resources/robots/biped/pm01/urdf/pm01_simple_collision.urdf (robot description, URDF)
Before this commit: robot pm01, 25 links, 24 joints
Joints:
- joint j02_hip_yaw_l: limit lower=-1.57 upper=4.014 effort=61 velocity=35.2 -> lower=-1.57 upper=4.014 effort=52 velocity=35.2
- joint j04_ankle_pitch_l: limit lower=-0.6807 upper=0.7243 effort=61 velocity=35.2 -> lower=-0.6807 upper=0.7243 effort=52 velocity=35.2
- joint j05_ankle_roll_l: limit lower=-0.2618 upper=0.2618 effort=61 velocity=35.2 -> lower=-0.2618 upper=0.2618 effort=52 velocity=35.2
- joint j08_hip_yaw_r: limit lower=-4.014 upper=1.57 effort=61 velocity=35.2 -> lower=-4.014 upper=1.57 effort=52 velocity=35.2
- joint j10_ankle_pitch_r: limit lower=-0.6807 upper=0.7243 effort=61 velocity=35.2 -> lower=-0.6807 upper=0.7243 effort=52 velocity=35.2
- joint j11_ankle_roll_r: limit lower=-0.2618 upper=0.2618 effort=61 velocity=35.2 -> lower=-0.2618 upper=0.2618 effort=52 velocity=35.2
- joint j12_waist_yaw: limit lower=-4.014 upper=1.57 effort=61 velocity=35.2 -> lower=-4.014 upper=1.57 effort=52 velocity=35.2
- joint j13_shoulder_pitch_l: limit lower=-2.9671 upper=2.7925 effort=61 velocity=35.2 -> lower=-2.9671 upper=2.7925 effort=52 velocity=35.2
- joint j14_shoulder_roll_l: limit lower=-0.6108 upper=2.3562 effort=61 velocity=35.2 -> lower=-0.6108 upper=2.3562 effort=52 velocity=35.2
- joint j15_shoulder_yaw_l: limit lower=-2.618 upper=2.618 effort=61 velocity=35.2 -> lower=-2.618 upper=2.618 effort=52 velocity=35.2
- joint j16_elbow_pitch_l: limit lower=-2.1948 upper=0.7374 effort=61 velocity=35.2 -> lower=-2.1948 upper=0.7374 effort=52 velocity=35.2
- joint j17_elbow_yaw_l: limit lower=-2.618 upper=2.618 effort=61 velocity=35.2 -> lower=-2.618 upper=2.618 effort=52 velocity=35.2
- joint j18_shoulder_pitch_r: limit lower=-2.9671 upper=2.7925 effort=61 velocity=35.2 -> lower=-2.9671 upper=2.7925 effort=52 velocity=35.2
- joint j19_shoulder_roll_r: limit lower=-2.3562 upper=0.6108 effort=61 velocity=35.2 -> lower=-2.3562 upper=0.6108 effort=52 velocity=35.2
- joint j20_shoulder_yaw_r: limit lower=-2.618 upper=2.618 effort=61 velocity=35.2 -> lower=-2.618 upper=2.618 effort=52 velocity=35.2
- joint j21_elbow_pitch_r: limit lower=-2.1948 upper=0.7374 effort=61 velocity=35.2 -> lower=-2.1948 upper=0.7374 effort=52 velocity=35.2
- joint j22_elbow_yaw_r: limit lower=-2.618 upper=2.618 effort=61 velocity=35.2 -> lower=-2.618 upper=2.618 effort=52 velocity=35.2
- joint j23_head_yaw: limit lower=-0.6109 upper=0.6109 effort=61 velocity=35.2 -> lower=-0.6109 upper=0.6109 effort=52 velocity=35.2
